File: ArduSatPowerSupplyModule.sch (EAGLE design)
At the start: 130 parts, among them IC10 ATMEGA32U4-QFN, IC11 MAX4372F, IC18 TMP102, IC19 TMP102, IC3 MAX17043G+U, IC7 MAX4372F, J1 POWER_JACKPTH, Q1 RJU003N03 N-MOSFET, Q2 MOSFET-PCHANNELSMT2, Q3 BSS138 N-MOSFET, Q4 BSS138 N-MOSFET, Q43 RJU003N03 N-MOSFET, Q44 RJU003N03 N-MOSFET, Q45 RJU003N03 N-MOSFET, Q46 RJU003N03 N-MOSFET, Q5 RJU003N03 N-MOSFET, SW1 SWITCH-DPDT2, SW2 RESET

Commit message: Totally restructured project: single 18650 cell; 0402 parts; shield footprint; dual MCUs in Eleven architecture
Parts:
- removed IC10: ATMEGA32U4-QFN, freetronics-jon:ATMEGA32U4-QFN
- removed JP8: M14SURFACE, freetronics-jon:M14SURFACE
- removed R15, R16: 4K7 0603, freetronics-master-v1.1:RESISTOR0603
- removed S4: (no value), freetronics-master-v1:M02PTH
- removed SW1: SWITCH-DPDT2, freetronics-jon:SWITCH-DPDT2
- added C31, C32: 22pF 0603, freetronics-jon:C-EU0402C
- added C35: 100nF 0402, freetronics-jon:C-EU0402C
- added C41: 100nF 0603, freetronics-jon:C-EU0402C
- added C43: 1uF 0603, freetronics-jon:C-EU0402C
- added CD: M01PTH, freetronics-2:M01PTH
- added IC1: AVR-MEGA8-MI, freetronics-jon:AVR-MEGA8-MI
- added IC8: ATMEGA16U2-MU, freetronics-jon:ATMEL_ATMEGA8U2-MUQFN
- added JP3: M100.1, freetronics-marc:M100.1
- added JP4, JP6: (no value), freetronics-marc:M08
- added JP9: (no value), freetronics-marc:M06SIP
- added L4: 0805 INDUCTOR, freetronics-master-v1:INDUCTOR0805-LARGE
- added P3: ICSP:USB, pinhead:PINHD-2X3
- added P4: microSD, freetronics-master-v1:USD-SOCKETNEW
- added R40, R49: 10K 0402, freetronics-jon:RESISTOR0402
- added R41: 4K7 0402, freetronics-jon:RESISTOR0402
- added R42, R45: 1M 0402, freetronics-jon:RESISTOR0402
- added R43, R44: 1K 0402, freetronics-jon:RESISTOR0402
- added RN6: 1K, freetronics-master-v1:4R-NCAY16
- added RN8: 2K2, freetronics-master-v1:4R-NCAY16
- added SJ10: USB_I, freetronics-jon:SJCN
- added SJ11: UGND, freetronics-jon:SJC0402
- added SJ6: RESET-EN, freetronics-jon:SJC0402
- added SJ7: 3V3_EN, freetronics-jon:SJCN
- added SJ8: UBOOT, freetronics-jon:SJ0402O
- added SJ9: DC_I, freetronics-jon:SJCN
- added U$14, U$20, U$21, U$23, U$24, U$25, U$26, U$3: SJCN, freetronics-jon:SJCN
- added U$27: CELLHOLDER-PCB, freetronics-jon:CELLHOLDER-PCB
- added U$28, U$29: FIDUCIAL1X2.5, freetronics-original:FIDUCIAL1X2.5
- added U$9: SWITCH-SPDT, freetronics-jon:SWITCH-SPDT
- added XTL2: 16MHz, freetronics-jon:CRYSTAL-GND3X2
- C1, C2: device SparkFun:CAP0402-CAP -> freetronics-jon:C-EU0402C
- C10: value 3300pF 0603 -> 3300pF 0402; device freetronics-master-v1.1:CAP0603 -> freetronics-jon:C-EU0402C
- C11, C6, C8: value 100nF 0603 -> 100nF 0402; device freetronics-master-v1.1:CAP0603 -> freetronics-jon:C-EU0402C
- C12: device freetronics-master-v1.1:CAP0603 -> freetronics-jon:C-EU0402C
- C13: value 1uF 0603 -> 100nF 0402; device freetronics-master-v1.1:CAP0603 -> freetronics-jon:C-EU0402C
- C14, C15: value 15pF 0603 -> 15pF 0402; device freetronics-master-v1.1:CAP0603 -> freetronics-jon:C-EU0402C
- C24: value 27pF 0603 -> 27pF 0402; device freetronics-master-v1.1:CAP0603 -> freetronics-jon:C-EU0402C
- C28: value 82pF 0603 -> 82pF 0402; device freetronics-master-v1.1:CAP0603 -> freetronics-jon:C-EU0402C
- JP5: value ICSP -> ICSP:MAIN
- JP7: value M14SURFACE -> (none); device freetronics-jon:M14SURFACE -> freetronics-marc:M02PTH
- LED1: value RED 0603 -> RED 0402; device freetronics-master-v1:LED0603 -> freetronics-jon:LED0402
- LED2: value BLUE 0603 -> BLUE 0402; device freetronics-master-v1:LED0603 -> freetronics-jon:LED0402
- LED4, LED5: device freetronics-master-v1:LED0603 -> freetronics-jon:LED0402
- Q3, Q4: value BSS138 N-MOSFET -> RJU003N03 N-MOSFET
- R1, R10, R11, R2, R22, R23, R3, R4, R5, R6, R7, R8, R9: device freetronics-master-v1.1:RESISTOR0603 -> freetronics-jon:RESISTOR0402
- R12: value 121K 1% 0603 -> 121K 1% 0402; device freetronics-master-v1.1:RESISTOR0603 -> freetronics-jon:RESISTOR0402
- R14, R37: value 249K 1% 0603 -> 249K 1% 0402; device freetronics-master-v1.1:RESISTOR0603 -> freetronics-jon:RESISTOR0402
- R19: value 10K 0603 -> 4K7 0402; device freetronics-master-v1.1:RESISTOR0603 -> freetronics-jon:RESISTOR0402
- R20, R21: value 10K 0603 -> 10K 0402
- R35: value 1M 1% 0603 -> 1M 1% 0402; device freetronics-master-v1.1:RESISTOR0603 -> freetronics-jon:RESISTOR0402
- R36: value 93.1K 1% 0603 -> 93.1K 1% 0402; device freetronics-master-v1.1:RESISTOR0603 -> freetronics-jon:RESISTOR0402
- S1: value USBSF-MICROB -> USB-6PSMT; device freetronics-jon:USBSF-MICROB -> freetronics-jon:USB-6PSMT
- SJ1, SJ2, SJ4, SJ5: device freetronics-master-v1:SJTINY -> freetronics-master-v1.1:SJ
- SJ3: value HWB -> 5V_EN; device freetronics-master-v1:SJTINY -> freetronics-jon:SJCN
- U$10: value CELLHOLDER2 -> FIDUCIAL1X2.5; device freetronics-jon:CELLHOLDER2 -> freetronics-original:FIDUCIAL1X2.5
Connections:
- removed net 3V3: C13.2, IC10.UCAP
- removed net A4: IC10.PF1(ADC1), JP8.2
- removed net A5: IC10.PF0(ADC0), JP8.1
- removed net D10_A11: IC10.PB6(OC1B/!OC4B!/ADC13), JP7.11
- removed net D11: IC10.PB7(OC0A/OC1C/RTS), JP7.12
- removed net D12: IC10.PD6(T1/OC4D/ADC9), JP7.13
- removed net D13: IC10.PC7(ICP3/CLK0/OC4A), JP7.14, RN2C.1
- removed net D4_A6: IC10.PD4(ICP1/ADC8), JP7.5
- removed net D6_A8: IC10.PD7(OC4D/ADC10/T0), JP7.7
- removed net D7_AIN0: IC10.PE6, JP7.8
- removed net D8_A9: IC10.PB4(ADC11), JP7.9
- removed net D9_A10: IC10.PB5(OC1A/!OC4B!/ADC12), JP7.10
- removed net H1L51: H1.51
- removed net H1R52: H1.52
- removed net MISO: IC10.PB3(PDO/MISO), JP5.1
- removed net MOSI: IC10.PB2(PDI/MOSI), JP5.4
- removed net RXLED_SS: IC10.PB0(SS), LED3.C-G
- removed net SCK: IC10.PB1(SCK), JP5.3
- removed net TX_LED: IC10.PD5(XCK/CTS), LED3.C-R
- new net +3V3_AS: H1.52, SJ7.2
- new net +5V_AS: H1.51, SJ3.2
- new net A4_SDA: IC1.PC4(ADC4/SDA), JP3.9, JP9.5, U$26.1
- new net A5_SCL: IC1.PC5(ADC5/SCL), JP3.10, JP9.6, U$25.1
- new net A6: IC1.ADC6, JP7.1
- new net A7: IC1.ADC7, JP7.2
- new net D10: IC1.PB2(SS/OC1B), JP3.3
- new net D11_MOSI: IC1.PB3(MOSI/OC2), JP3.4, JP5.4, RN6C.2
- new net D12_MISO: IC1.PB4(MISO), JP3.5, JP5.1, P4.DO
- new net D13_SCK: IC1.PB5(SCK), JP3.6, JP5.3, RN2C.1, RN6B.2
- new net D4: IC1.PD4(XCK/T0), JP4.5, RN6D.2
- new net D6: IC1.PD6(AIN0), JP4.7
- new net D7: IC1.PD7(AIN1), JP4.8
- new net D8: IC1.PB0(ICP), JP3.1
- new net D9: IC1.PB1(OC1A), JP3.2
- new net DC_I: R5.1, SJ9.1, U$19.IDC
- new net DTR: IC8.(CTS)PD7, SJ6.1, SJ8.2
- new net MISO2: IC8.(MISO)PB3, P3.1
- new net MOSI2: IC8.(MOSI)PB2, P3.4
- new net N$13: P4.CS, RN6D.1, RN8A.2
- new net N$24: C32.2, IC1.PB7(XTAL2/TOSC2), R42.1, XTL2.XTL1
- new net N$34: C43.1, IC8.UCAP
- new net N$38: C12.2, L4.2, S1.FIX1, S1.FIX2, S1.PIN1, S1.PIN2, S1.TAB1, S1.TAB2, Z1.1, Z2.1, Z3.A
- new net N$46: P4.DI, RN6C.1, RN8C.2
- new net N$48: P4.SCK, RN6B.1, RN8B.2
- new net N$50: CD.1, P4.CD1
- new net N$51: IC7.OUT, U$14.1
- new net N$52: C14.2, IC8.XTAL2, R45.2, XTL1.XTL2
- new net N$53: IC18.V+, Q43.G, Q44.G, R83.2, R84.2, U$23.2
- new net N$54: IC19.ADD0, IC19.V+, Q45.G, Q46.G, R85.2, R86.2, U$24.2
- new net N$55: Q3.S, R20.1, U$25.2
- new net N$56: IC8.UGND, L4.1, S1.GND, SJ11.1
- new net N$57: Q4.S, R21.1, U$26.2
- new net N$60: C35.1, SJ6.2
- new net NC: JP6.1
- new net RESET2: IC8.RESET, P3.5, R49.1
- new net RXLED: IC8.PD4, LED3.C-G
- new net SCK2: IC8.(SCLK)PB1, P3.3
- new net SYS_SCL: H1.43, U$21.2
- new net SYS_SDA: H1.41, U$20.2
- new net TXLED: IC8.(XCK)PD5, LED3.C-R
- new net USBRXD: IC8.(TXD1)PD3, R44.2
- new net USBTXD: IC8.(RXD1)PD2, R43.2
- new net USB_I: R6.1, SJ10.1, U$19.IUSB
- net +5V_SYS: no longer R15.2, R16.2
- net 3.3V: now also C13.1, JP6.4, P4.VCC, SJ7.1, U$23.1, U$24.1; no longer IC18.V+, IC19.ADD0, IC19.V+, JP8.11, Q43.G, Q44.G, Q45.G, Q46.G, R83.2, R84.2, R85.2, R86.2
- net 5V: now also IC1.AVCC, IC1.VCC@1, IC1.VCC@2, JP6.2, JP6.5, R19.2, R40.2, R41.2, SJ3.1; no longer IC10.AVCC, IC10.AVCC1, IC10.VCC, IC10.VCC1, JP8.10, JP8.13, R19.1, RN2A.1, RN2B.1
- net A0: now also IC1.PC0(ADC0), JP9.1, SJ9.2; no longer IC10.PF7(ADC7(TDI), JP8.6, R5.1, U$19.IDC
- net A1: now also IC1.PC1(ADC1), JP9.2, SJ10.2; no longer IC10.PF6(ADC6/TDO), JP8.5, R6.1, U$19.IUSB
- net A2: now also IC1.PC2(ADC2), JP9.3, U$14.2; no longer IC10.PF5(ADC5/TMS), IC11.OUT, JP8.4
- net A3: now also IC1.PC3(ADC3), JP9.4, U$3.2; no longer IC10.PF4(ADC4/TCK), IC7.OUT, JP8.3
- net AREF: now also IC1.AREF, JP3.8; no longer IC10.AREF, JP8.14
- net BAT: now also U$27.+, U$9.1; no longer S4.1, SW1.2, SW1.5
- net D0_RX: now also IC1.PD0(RXD), JP4.1, R44.1; no longer IC10.PD2(INT2/RXD1), JP7.1
- net D1_TX: now also IC1.PD1(TXD), JP4.2, R43.1; no longer IC10.PD3(INT3/TXD1), JP7.2
- net D2_SDA: now also IC1.PD2(INT0), JP4.3; no longer IC10.PD1(INT1/SDA), JP7.3, Q4.S, R21.1
- net D3_SCL: now also IC1.PD3(INT1), JP4.4; no longer IC10.PD0(INT0/OC0B/SCL), JP7.4, Q3.S, R20.1
- net D5: now also IC1.PD5(T1), JP4.6; no longer IC10.PC6(OC3A/!OC4A!), JP7.6
- net GND: now also C13.2, C31.1, C32.1, C41.2, C43.2, IC1.AGND, IC1.GND@1, IC1.GND@2, IC1.TGND, IC8.GND, IC8.PAD, JP3.7, JP6.6, JP6.7, P3.6, P4.CD2, P4.GND, P4.SHIELD1, P4.SHIELD2, RN8A.1, RN8B.1, RN8C.1, SJ11.2, SJ8.1, U$27.-, XTL2.GND, XTL2.GND2; no longer C12.2, C13.1, IC10.GND, IC10.GND1, IC10.GND2, IC10.GND3, IC10.TGND, IC10.UGND, JP8.8, JP8.9, S1.FIX1, S1.FIX2, S1.GND, S1.TAB1, S1.TAB2, S4.2, SJ3.2, Z1.1, Z2.1, Z3.A
- net N$10: now also C31.2, IC1.PB6(XTAL1/TOSC1), R42.2, XTL2.XTL2; no longer IC10.PE2(HWB), SJ3.1
- net N$11: now also IC11.OUT, U$3.1; no longer C14.2, IC10.XTAL1, XTL1.XTL2
- net N$12: now also IC8.XTAL1, R45.1; no longer IC10.XTAL2
- net N$5: now also U$9.2; no longer SW1.3, SW1.4
- net PVIN: now also JP6.8
- net RD+: now also IC8.D+; no longer IC10.D+
- net RD-: now also IC8.D-; no longer IC10.D-
- net RESET: now also C35.2, IC1.PC6(/RESET), JP6.3, R40.1; no longer IC10./RESET, JP8.12, R19.2
- net SCL: now also R41.1, U$21.1; no longer H1.43, R16.1
- net SDA: now also R19.1, U$20.1; no longer H1.41, R15.1
- net USBVCC: now also C41.1, IC8.AVCC, IC8.UVCC, IC8.VCC, P3.2, R49.2, RN2A.1, RN2B.1; no longer IC10.UVCC, IC10.VBUS, JP8.7
Other:
- note added: "ATmega16U2 Microcontroller"
- note added: "ATmega328P Microcontroller"
- note added: "I2C Pullups And Isolation"
- note added: "ICSP"
- note added: "SJ3 shorted by default SJ4 open by default"
- note added: "SJ7 shorted by default SJ5 open by default"
- note added: "V1.0 (2013-02-24)"
- note added: "micro SD Card Slot"
- note added: "uSD_nCS"
- note removed: "(Not fitted)"
- note removed: "ATmega32u4 MCU"
- note removed: "Connect across SJ3 after other routing"
- note removed: "Short across SJ4 after other routing"
- note removed: "Short across SJ5 after other routing"
- note removed: "System I2C Pullups"
- note removed: "V1.0 (2013-01-14)"
- note removed: "~"

Commit message: Routing done, clearances, DRC, overlay. Nearly ready for v1.0 release
Parts:
- removed C61: 100nF 0402, freetronics-jon:C-EU0402C
- removed IC19: TMP102, freetronics-jon:TMP102
- removed P3: ICSP:USB, pinhead:PINHD-2X3
- removed P4: microSD, freetronics-master-v1:USD-SOCKETNEW
- removed R49, R84: 10K 0402, freetronics-jon:RESISTOR0402
- removed RN8: 2K2, freetronics-master-v1:4R-NCAY16
- removed U$11: LTC3115, freetronics-jon:LTC3115
- removed U$15: LTC3536, freetronics-jon:LTC3536
- removed U$9: SWITCH-SPDT, freetronics-jon:SWITCH-SPDT
- added C30: 22pF 0402, freetronics-jon:C-EU0402C
- added IC2: ATMEGA16U2-MU, freetronics-jon:ATMEL_ATMEGA8U2-MUQFN
- added IC5: MAX17043G+U, SparkFun:MAX1704X
- added IC6: MAX4372F, freetronics-jon:MAX4372
- added JP10, JP11: (no value), freetronics-master-v1:M02PTH
- added R15: 121K 1% 0402, freetronics-jon:RESISTOR0402
- added R16: 93.1K 1% 0402, freetronics-jon:RESISTOR0402
- added RN1: 1K5, resistor-dil:4R-NCAY16
- added SW1: RESET, freetronics-master-v1:TAC_SWITCH_2PIN
- C19: value 1nF -> 1nF 0402
- C2: value 10nF -> 10nF 0402
- C21, C33, C7: value 100nF 0603 -> 100nF 0402
- C26: value 100pF -> 100pF 0402
- C31: value 22pF 0603 -> 22pF 0402
- C32: value 22pF 0603 -> 100nF 0402
- IC11: value MAX4372F -> TMP102; device freetronics-jon:MAX4372 -> freetronics-jon:TMP102
- IC3: value MAX17043G+U -> LTC3115; device SparkFun:MAX1704X -> freetronics-jon:LTC3115
- IC7: value MAX4372F -> LTC3536; device freetronics-jon:MAX4372 -> freetronics-jon:LTC3536
- IC8: value ATMEGA16U2-MU -> MAX4372F; device freetronics-jon:ATMEL_ATMEGA8U2-MUQFN -> freetronics-jon:MAX4372
- JP1: value (none) -> ICSP:16U2; device freetronics-master-v1:M02PTH -> pinhead:PINHD-2X3
- JP2: value (none) -> ICSP:328P; device freetronics-master-v1:M02PTH -> pinhead:PINHD-2X3
- JP3: value M100.1 -> (none); device freetronics-marc:M100.1 -> freetronics-marc:M08
- JP4: device freetronics-marc:M08 -> freetronics-marc:M06SIP
- JP5: value ICSP:MAIN -> (none); device pinhead:PINHD-2X3 -> freetronics-marc:M02PTH
- JP6: value (none) -> M100.1; device freetronics-marc:M08 -> freetronics-marc:M100.1
- JP7: device freetronics-marc:M02PTH -> freetronics-marc:M08
- JP8: value M01PTH -> CD
- JP9: device freetronics-marc:M06SIP -> freetronics-master-v1:M02PTH
- LED4: value BLUE -> BLUE 0402
- LED5: value JADEGREEN -> JADEGREEN 0402
- Q2: value MOSFET-PCHANNELSMT2 -> RJU003N03 N-MOSFET; device freetronics-jon:MOSFET-PCHANNELSMT2 -> freetronics-jon:MOSFET-NSOT-323
- Q3: value RJU003N03 N-MOSFET -> MOSFET-PCHANNELSMT2; device freetronics-jon:MOSFET-NSOT-323 -> freetronics-jon:MOSFET-PCHANNELSMT2
- R1: value 1K -> 1M 0402
- R10: value 33K -> 10K 0402
- R11: value 1K -> 2K2 0402
- R12: value 121K 1% 0402 -> 1K 0402
- R13: value 0.1R 2010 -> 4K7 0402; device freetronics-original:RESISTOR2010 -> freetronics-jon:RESISTOR0402
- R14: value 249K 1% 0402 -> 4K7 0402
- R17: value 10K 0402 -> 1M 1% 0402
- R18: value 10K 0402 -> 249K 1% 0402
- R19: value 4K7 0402 -> 249K 1% 0402
- R2: value 4K7 -> 10K 0402
- R20: value 10K 0402 -> 1K
- R21: value 10K 0402 -> 1.05K 1% 0603
- R22: value 2K2 -> 1.18K 1% 0603
- R23: value 1K -> 1K 1% 0402
- R24: value 49.9K -> 10K 0603
- R25: value 187K -> 2K2 0402
- R26: value 100K -> 1K 0402
- R27: value 845K -> 1K
- R28: value 15K -> 33K
- R29: value 0.1R 2010 -> 1K 0402; device freetronics-original:RESISTOR2010 -> freetronics-jon:RESISTOR0402
- R3: value 2K2 -> 22R
- R30: value 49.9K -> 4K7 0402
- R31: value 115K -> 10K 0402
- R32: value 100K -> 10K 0402
- R33: value 845K -> 0.1R 2010; device freetronics-jon:RESISTOR0402 -> freetronics-original:RESISTOR2010
- R34: value 15K -> 100K
- R35: value 1M 1% 0402 -> 49.9K
- R36: value 93.1K 1% 0402 -> 15K 0402
- R37: value 249K 1% 0402 -> 115K 1% 0402
- R38: value 22R -> 845K 1% 0402
- R39: value 22R -> 0.1R 2010; device freetronics-jon:RESISTOR0402 -> freetronics-original:RESISTOR2010
- R4: value 1K 1% 0603 -> 22R
- R40: value 10K 0402 -> 100K
- R41: value 4K7 0402 -> 49.9K 1% 0402
- R42: value 1M 0402 -> 15K
- R43: value 1K 0402 -> 187K 1% 0402
- R44: value 1K 0402 -> 845K 1% 0402
- R45: value 1M 0402 -> 10K 0402
- R5: value 1.05K 1% 0603 -> 1M 0402
- R6: value 1.18K 1% 0603 -> 10K 0402
- R7: value 1K -> 1K 0402
- R8: value 10K 0603 -> 1K 0402
- R9: value 1K -> 10K 0402
- RN2: value 1K5 -> 2K2; device resistor-dil:4R-NCAY16 -> freetronics-master-v1:4R-NCAY16
- S2: value (none) -> microSD; device freetronics-master-v1:M02PTH -> freetronics-master-v1:USD-SOCKETNEW
- SW2: value RESET -> SWITCH-SPDT; device freetronics-master-v1:TAC_SWITCH_2PIN -> freetronics-jon:SWITCH-SPDT
- renumbered C41 to C33, C43 to C34, C62 to C36, CD to JP8, IC18 to IC10, J1 to S3, Q43 to Q6, Q44 to Q7, Q45 to Q8, Q46 to Q9, R83 to R46, R85 to R48, R86 to R47, RN6 to RN3, U$12 to IC9, U$14 to SJ19, U$19 to IC4, U$20 to SJ12, U$21 to SJ13, U$23 to SJ14, U$24 to SJ15, U$25 to SJ16, U$26 to SJ17, U$27 to BAT1, U$3 to SJ18
Connections:
- net 3.3V: now also C35.1, IC5.VDD, JP3.4, Q4.G, R12.1, R31.2, R32.2, R42.2, R44.2, S2.VCC; no longer C61.1, IC3.VDD, JP6.4, P4.VCC, Q1.G, R17.2, R18.2, R23.1, R27.2, R28.2
- net 3V3SENSED: now also IC8.RS-, IC8.VCC, R39.2; no longer IC7.RS-, IC7.VCC, R13.2
- net 5V: now also IC7.VOUT, JP2.2, JP3.2, JP3.5, Q1.G, Q2.G, R10.2, R11.1, R13.2, R14.2, R36.2, R38.2, R6.2, R9.2; no longer JP5.2, JP6.2, JP6.5, Q3.G, Q4.G, R19.2, R20.2, R21.2, R22.1, R33.2, R34.2, R40.2, R41.2, U$15.VOUT
- net 5VSENSED: now also IC6.RS-, IC6.VCC, IC7./SHDN, IC7.VIN, R33.2; no longer IC11.RS-, IC11.VCC, R29.2, U$15./SHDN, U$15.VIN
- net A0: now also JP4.1; no longer JP9.1
- net A1: now also JP4.2; no longer JP9.2
- net A2: now also JP4.3; no longer JP9.3
- net A3: now also JP4.4; no longer JP9.4
- net A4_SDA: now also JP4.5, JP6.9; no longer JP3.9, JP9.5
- net A5_SCL: now also JP4.6, JP6.10; no longer JP3.10, JP9.6
- net A6: now also JP5.1; no longer JP7.1
- net A7: now also JP5.2; no longer JP7.2
- net AREF: now also JP6.8; no longer JP3.8
- net BAT: now also R25.1, R26.1, R29.2, SW2.1; no longer R1.2, R3.1, R7.1, U$9.1
- net CELL: now also IC5.CELL, R29.1; no longer IC3.CELL, R1.1
- net D+: now also R4.1; no longer R39.1
- net D-: now also R3.1; no longer R38.1
- net D0_RX: now also JP7.1, R8.1; no longer JP4.1, R44.1
- net D10: now also JP6.3; no longer JP3.3
- net D11_MOSI: now also JP2.4, JP6.4; no longer JP3.4, JP5.4
- net D12_MISO: now also JP2.1, JP6.5, S2.DO; no longer JP3.5, JP5.1, P4.DO
- net D13_SCK: now also JP2.3, JP6.6, RN1C.1; no longer JP3.6, JP5.3, RN2C.1
- net D1_TX: now also JP7.2, R7.1; no longer JP4.2, R43.1
- net D2_SDA: now also JP7.3; no longer JP4.3
- net D3_SCL: now also JP7.4; no longer JP4.4
- net D4: now also JP7.5; no longer JP4.5
- net D5: now also JP7.6; no longer JP4.6
- net D6: now also JP7.7; no longer JP4.7
- net D7: now also JP7.8; no longer JP4.8
- net D8: now also JP6.1; no longer JP3.1
- net D9: now also JP6.2; no longer JP3.2
- net DC_I: now also R21.1; no longer R5.1
- net DTR: now also IC2.(CTS)PD7; no longer IC8.(CTS)PD7
- net GND: now also C30.1, C35.2, IC2.GND, IC2.PAD, IC3.GND1, IC3.GND2, IC3.PGND, IC5.CTG, IC5.GND@4, IC5.GND@EP, IC6.GND, IC7.MODE/SYNC, IC7.SGND, IC7.TGND, JP1.6, JP10.1, JP2.6, JP3.6, JP9.1, R15.1, R18.1, R21.2, R22.2, R23.2, R24.2, R30.1, R34.2, R37.2, R40.2, R43.2, RN2A.1, RN2B.1, RN2C.1, S2.CD2, S2.GND, S2.SHIELD1, S2.SHIELD2, SW1.P; no longer C32.1, C61.2, IC19.GND, IC3.CTG, IC3.GND@4, IC3.GND@EP, IC7.GND, IC8.PAD, JP1.1, JP5.6, JP6.6, P3.6, P4.CD2, P4.GND, P4.SHIELD1, P4.SHIELD2, R12.1, R14.1, R2.1, R25.2, R26.2, R31.2, R32.2, R4.2, R5.2, R6.2, R8.2, RN8A.1, RN8B.1, RN8C.1, S2.1, SW2.P, U$11.GND1, U$11.GND2, U$11.PGND, U$15.MODE/SYNC, U$15.SGND, U$15.TGND
- net MISO2: now also IC2.(MISO)PB3, JP1.1; no longer IC8.(MISO)PB3, P3.1
- net MOSI2: now also IC2.(MOSI)PB2, JP1.4; no longer IC8.(MOSI)PB2, P3.4
- net N$1: now also R12.2; no longer R23.2
- net N$10: now also C30.2, R5.2; no longer C31.2, R42.2
- net N$10001: now also R45.1; no longer R84.1
- net N$10002: now also IC11.SDA; no longer IC19.SDA
- net N$10003: now also IC11.SCL; no longer IC19.SCL
- net N$11: now also IC6.OUT; no longer IC11.OUT
- net N$12: now also IC2.XTAL1, R1.1; no longer IC8.XTAL1, R45.1
- net N$13: now also RN2A.2, S2.CS; no longer P4.CS, RN8A.2
- net N$14: now also RN1C.2; no longer RN2C.2
- net N$15: now also R41.1; no longer R24.1
- net N$16: now also RN1B.2; no longer RN2B.2
- net N$17: now also RN1A.2; no longer RN2A.2
- net N$2: now also JP10.2, JP11.1; no longer JP1.2, JP2.1
- net N$20: now also R24.1; no longer R8.1
- net N$21: now also R40.1; no longer R26.1
- net N$22: now also IC7.SW1; no longer U$15.SW1
- net N$23: now also R41.2; no longer R24.2
- net N$24: now also C31.2, R5.1; no longer C32.2, R42.1
- net N$248: now also R26.2; no longer R7.2
- net N$25: now also R42.1; no longer R28.1
- net N$26: now also R43.1, R44.1; no longer R25.1, R27.1
- net N$28: now also IC7.SW2; no longer U$15.SW2
- net N$29: now also IC7.RT, R34.1; no longer R32.1, U$15.RT
- net N$3: now also R25.2; no longer R3.2
- net N$30: now also R35.2; no longer R30.2
- net N$31: now also IC7.VC, R35.1; no longer R30.1, U$15.VC
- net N$32: now also R36.1; no longer R34.1
- net N$33: now also IC7.FB, R37.1, R38.1; no longer R31.1, R33.1, U$15.FB
- net N$34: now also IC2.UCAP; no longer IC8.UCAP
- net N$35: now also R23.1; no longer R4.1
- net N$36: now also R20.2; no longer R11.2
- net N$37: now also R16.2; no longer R36.2
- net N$39: now also IC3.PVCC, IC3.PWM/SYNC, IC3.VCC; no longer U$11.PVCC, U$11.PWM/SYNC, U$11.VCC
- net N$4: now also JP11.2, R27.1; no longer JP2.2, R9.1
- net N$40: now also IC3.BST1; no longer U$11.BST1
- net N$41: now also IC3.BST2; no longer U$11.BST2
- net N$42: now also IC3.SW1; no longer U$11.SW1
- net N$43: now also IC3.SW2; no longer U$11.SW2
- net N$44: now also IC3.VC, R16.1; no longer R36.1, U$11.VC
- net N$45: now also IC3.FB, R17.1, R18.2, R19.1; no longer R14.2, R35.1, R37.1, U$11.FB
- net N$46: now also RN2C.2, S2.DI; no longer P4.DI, RN8C.2
- net N$47: now also IC3.RT, R15.2; no longer R12.2, U$11.RT
- net N$48: now also RN2B.2, S2.SCK; no longer P4.SCK, RN8B.2
- net N$49: now also R19.2; no longer R37.2
- net N$5: now also Q3.S, R28.1, SW2.2; no longer Q2.S, R10.1, U$9.2
- net N$50: now also S2.CD1; no longer P4.CD1
- net N$51: now also IC8.OUT; no longer IC7.OUT
- net N$52: now also IC2.XTAL2, R1.2; no longer IC8.XTAL2, R45.2
- net N$53: now also R45.2; no longer R84.2
- net N$54: now also IC11.ADD0, IC11.V+; no longer IC19.ADD0, IC19.V+
- net N$55: now also Q1.S, R9.1; no longer Q3.S, R20.1
- net N$56: now also IC2.UGND; no longer IC8.UGND
- net N$57: now also Q2.S, R10.1; no longer Q4.S, R21.1
- net N$6: now also R11.2; no longer R22.2
- net N$60: now also C32.1; no longer C35.1
- net N$7: now also Q3.G, R27.2, R28.2; no longer Q2.G, R10.2, R9.2
- net N$8: now also IC5.SDA, Q4.S, R32.1; no longer IC3.SDA, Q1.S, R17.1
- net N$9: now also IC5.SCL, R31.1; no longer IC3.SCL, R18.1
- net NC: now also JP3.1; no longer JP6.1
- net PVIN: now also IC3.PVIN, IC3.RUN, IC3.VIN, JP3.8, JP9.2; no longer JP6.8, S2.2, U$11.PVIN, U$11.RUN, U$11.VIN
- net PVOUT: now also IC3.PVOUT, R17.2; no longer R35.2, U$11.PVOUT
- net QST: now also IC5.QST, R30.2; no longer IC3.QST, R2.2
- net RD+: now also IC2.D+, R4.2; no longer IC8.D+, R39.2
- net RD-: now also IC2.D-, R3.2; no longer IC8.D-, R38.2
- net RESET: now also C32.2, JP2.5, JP3.3, R6.1, SW1.S; no longer C35.2, JP5.5, JP6.3, R40.1, SW2.S
- net RESET2: now also IC2.RESET, JP1.5, R2.1; no longer IC8.RESET, P3.5, R49.1
- net RXLED: now also IC2.PD4; no longer IC8.PD4
- net SCK2: now also IC2.(SCLK)PB1, JP1.3; no longer IC8.(SCLK)PB1, P3.3
- net SCL: now also Q1.D, R13.1; no longer Q3.D, R41.1
- net SDA: now also Q2.D, R14.1; no longer Q1.D, R19.1
- net TXLED: now also IC2.(XCK)PD5; no longer IC8.(XCK)PD5
- net USBRXD: now also IC2.(TXD1)PD3, R8.2; no longer IC8.(TXD1)PD3, R44.2
- net USBTXD: now also IC2.(RXD1)PD2, R7.2; no longer IC8.(RXD1)PD2, R43.2
- net USBVCC: now also IC2.AVCC, IC2.UVCC, IC2.VCC, JP1.2, R2.2, R20.1, RN1A.1, RN1B.1; no longer IC8.AVCC, IC8.UVCC, IC8.VCC, P3.2, R11.1, R49.2, RN2A.1, RN2B.1
- net USB_I: now also R22.1; no longer R6.1
- net VBATT: now also IC6.RS+, IC8.RS+, Q3.D, R33.1, R39.1; no longer IC11.RS+, IC7.RS+, Q2.D, R13.1, R29.1
